Commit message: added meshes for visualisation in rviz

File: install/pick_place_arms/share/pick_place_arms/urdf/pick_place.urdf (robot description, URDF)
Before this commit: robot pick_place, 2 links, 1 joints
Links:
- added link arm_link, mass 3.0; collision cylinder length=0.2 radius=0.04; visual mesh filename=package://pick_place_arms/meshes/Shoulder_arm.stl scale=0.001 0.001 0.001
- added link shoulder_link, mass 5.0; collision cylinder length=0.2 radius=0.05; visual mesh filename=package://pick_place_arms/meshes/Shoulder.stl scale=0.001 0.001 0.001
- link base_link: geometry collision box size=0.4 0.2 0.1; visual mesh filename=package://pick_place_arms/meshes/Base.stl scale=0.001 0.001 0.001
Joints:
- added joint arm_joint: type revolute, parent base_link, child shoulder_link, origin xyz=0 0 0.1 rpy=0 0 0, axis 0 0 1, limit lower=-1.57 upper=1.57 effort=10 velocity=1.0
- added joint elbow_joint: type revolute, parent shoulder_link, child arm_link, origin xyz=0 0 0.2 rpy=0 0 0, axis 0 0 1, limit lower=-1.57 upper=1.57 effort=10 velocity=1.0

File: src/pick_place_arms/urdf/pick_place.urdf (robot description, URDF)
Before this commit: robot pick_place, 2 links, 0 joints
Links:
- added link arm_link, mass 3.0; collision cylinder length=0.2 radius=0.04; visual mesh filename=package://pick_place_arms/meshes/Shoulder_arm.stl scale=0.001 0.001 0.001
- added link shoulder_link, mass 5.0; collision cylinder length=0.2 radius=0.05; visual mesh filename=package://pick_place_arms/meshes/Shoulder.stl scale=0.001 0.001 0.001
- link base_link: geometry collision box size=0.4 0.2 0.1; visual mesh filename=package://pick_place_arms/meshes/Base.stl scale=0.001 0.001 0.001
Joints:
- added joint arm_joint: type revolute, parent base_link, child shoulder_link, origin xyz=0 0 0.1 rpy=0 0 0, axis 0 0 1, limit lower=-1.57 upper=1.57 effort=10 velocity=1.0
- added joint base_to_arm: type fixed, parent base_footprint, child base_link, origin xyz=0 0 0.05 rpy=0 0 0
- added joint elbow_joint: type revolute, parent shoulder_link, child arm_link, origin xyz=0 0 0.2 rpy=0 0 0, axis 0 0 1, limit lower=-1.57 upper=1.57 effort=10 velocity=1.0
