Commit message: worked on the origin of the meshes, figuring out each joint and origin

File: src/pick_place_arms/urdf/pick_place.urdf (robot description, URDF)
Before this commit: robot pick_place, 4 links, 3 joints
Joints:
- joint arm_joint: origin xyz=0 0 0.1 rpy=0 0 0 -> xyz=0 0 0.01 rpy=0 0 0
- joint base_to_arm: origin xyz=0 0 0.05 rpy=0 0 0 -> xyz=0 0 0 rpy=0 0 0
- joint elbow_joint: axis 0 0 1 -> 1 0 0; origin xyz=0 0 0.2 rpy=0 0 0 -> xyz=0 0 0 rpy=0 0 0

Commit message: I've completed visualisation on rviz

File: src/pick_place_arms/urdf/pick_place.urdf (robot description, URDF)
Before this commit: robot pick_place, 4 links, 3 joints
Links:
- added link gripper_left_finger_link, mass 0.2; collision box size=0.02 0.05 0.05; visual mesh filename=package://pick_place_arms/meshes/Left gripper.stl scale=0.0015 0.0015 0.0015
- added link gripper_link, mass 1.0; collision box size=0.1 0.1 0.1; visual mesh filename=package://pick_place_arms/meshes/arm.stl scale=0.0015 0.0015 0.0015
- added link gripper_right_finger_link, mass 0.2; collision box size=0.02 0.05 0.05; visual mesh filename=package://pick_place_arms/meshes/Right gripper.stl scale=0.0015 0.0015 0.0015
Joints:
- added joint gripper_joint: type revolute, parent arm_link, child gripper_link, origin xyz=0 0 0.0315 rpy=0 0 0, axis 1 0 0, limit lower=-1.57 upper=1.57 effort=10 velocity=1.0
- added joint gripper_left_finger_joint: type prismatic, parent gripper_link, child gripper_left_finger_link, origin xyz=0 0 0.03 rpy=0 0 0, axis 0 1 0, limit lower=-0.004 upper=-0 effort=100.0 velocity=4.0
- added joint gripper_right_finger_joint: type prismatic, parent gripper_link, child gripper_right_finger_link, origin xyz=0 0 0.03 rpy=0 0 0, axis 0 1 0, limit lower=0 upper=0.004 effort=5 velocity=1.0
- joint elbow_joint: origin xyz=0 0 0 rpy=0 0 0 -> xyz=0 0 0.015 rpy=0 0 0

Commit message: I've added an rqt tree

File: src/pick_place_arms/urdf/pick_place.urdf (robot description, URDF)
Before this commit: robot pick_place, 7 links, 6 joints
Joints:
- joint gripper_left_finger_joint: axis 0 1 0 -> 1 0 0; limit lower=-0.004 upper=-0 effort=100.0 velocity=4.0 -> lower=0.004 upper=0 effort=100.0 velocity=4.0
- joint gripper_right_finger_joint: axis 0 1 0 -> 1 0 0; limit lower=0 upper=0.004 effort=5 velocity=1.0 -> lower=0 upper=-0.004 effort=5 velocity=1.0

Commit message: I have added a joint state publisher and there is an error I'm trying to figure it out

File: src/pick_place_arms/urdf/pick_place.urdf (robot description, URDF)
Before this commit: robot pick_place, 7 links, 6 joints
Joints:
- removed joint base_to_arm
- added joint base_joint: type fixed, parent base_footprint, child base_link, origin xyz=0 0 0 rpy=0 0 0
- joint gripper_left_finger_joint: limit lower=0.004 upper=0 effort=100.0 velocity=4.0 -> lower=0 upper=0.004 effort=100.0 velocity=4.0
- joint gripper_right_finger_joint: limit lower=0 upper=-0.004 effort=5 velocity=1.0 -> lower=-0.004 upper=0 effort=5 velocity=1.0
